File: iot master.kicad_sch (KiCad schematic)
At the start: 0 parts

Commit message: Add files via upload
Changed lines of the file:
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@@
     )
   )
-  (sheet (at 77.47 54.61) (size 43.18 34.29) (fields_autoplaced)
+  (sheet (at 74.93 48.26) (size 43.18 34.29) (fields_autoplaced)
     (stroke (width 0) (type solid) (color 0 0 0 0))
     (fill (color 0 0 0 0.0000))
-    (property "Sheet name" "relays" (id 0) (at 77.47 53.5301 0)
+    (property "Sheet name" "relays" (id 0) (at 74.93 47.1801 0)
       (effects (font (size 2.0066 2.0066)) (justify left bottom))
     )
-    (property "Sheet file" "relays.kicad_sch" (id 1) (at 77.47 89.7792 0)
+    (property "Sheet file" "relays.kicad_sch" (id 1) (at 74.93 83.4292 0)
       (effects (font (size 2.0066 2.0066)) (justify left top))
     )
   )
-  (sheet (at 123.19 54.61) (size 46.99 34.29) (fields_autoplaced)
+  (sheet (at 120.65 48.26) (size 46.99 34.29) (fields_autoplaced)
     (stroke (width 0) (type solid) (color 0 0 0 0))
     (fill (color 0 0 0 0.0000))
-    (property "Sheet name" "maincontroller" (id 0) (at 123.19 53.5301 0)
+    (property "Sheet name" "maincontroller" (id 0) (at 120.65 47.1801 0)
       (effects (font (size 2.0066 2.0066)) (justify left bottom))
     )
-    (property "Sheet file" "maincontroller.kicad_sch" (id 1) (at 123.19 89.7792 0)
+    (property "Sheet file" "maincontroller.kicad_sch" (id 1) (at 120.65 83.4292 0)
       (effects (font (size 2.0066 2.0066)) (justify left top))
     )
@@
     )
     (path "/00000000-0000-0000-0000-000062edbe16/e76bc692-e02d-44b1-90d2-4ded5e4a7b61"
-      (reference "#PWR?") (unit 1) (value "GND") (footprint "")
+      (reference "#PWR0139") (unit 1) (value "GND") (footprint "")
     )
     (path "/00000000-0000-0000-0000-000062e8cfa7/00000000-0000-0000-0000-000062e9e0fd"
@@
     )
     (path "/00000000-0000-0000-0000-000062e8cfa7/00000000-0000-0000-0000-000062e9e15c"
-      (reference "R14") (unit 1) (value "120") (footprint "Resistor_SMD:R_0805_2012Metric_Pad1.15x1.40mm_HandSolder")
+      (reference "R14") (unit 1) (value "120NC") (footprint "Resistor_SMD:R_0805_2012Metric_Pad1.15x1.40mm_HandSolder")
     )
     (path "/00000000-0000-0000-0000-000062edbe16/00000000-0000-0000-0000-000062ef70b8"
