File: MAX485CIRCUIT.kicad_sch (KiCad schematic)
At the start: 16 parts, among them J1 Screw_Terminal_01x03, Q3 2N2219, U1 MAX485E

Commit message: Add files via upload
Parts:
- R14: value 120 -> 120NC
Other:
- note added: "the 120 should be connected at the master device and the last slave one"
Changed lines of the file:
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@@
   (junction (at 194.31 102.87) (diameter 0) (color 0 0 0 0)
   )
-  (junction (at 186.69 102.87) (diameter 0) (color 0 0 0 0)
-  )
   (junction (at 121.92 99.06) (diameter 0) (color 0 0 0 0)
   )
@@
   (junction (at 163.83 119.38) (diameter 0) (color 0 0 0 0)
   )
+  (junction (at 186.69 106.68) (diameter 0) (color 0 0 0 0)
+  )
   (junction (at 127 101.6) (diameter 0) (color 0 0 0 0)
   )
@@
     (stroke (width 0) (type default) (color 0 0 0 0))
   )
-  (wire (pts (xy 181.61 99.06) (xy 173.99 99.06))
-    (stroke (width 0) (type default) (color 0 0 0 0))
-  )
   (wire (pts (xy 72.39 99.06) (xy 72.39 95.25))
     (stroke (width 0) (type default) (color 0 0 0 0))
@@
     (stroke (width 0) (type default) (color 0 0 0 0))
   )
-  (wire (pts (xy 186.69 102.87) (xy 176.53 102.87))
-    (stroke (width 0) (type default) (color 0 0 0 0))
-  )
   (wire (pts (xy 81.28 101.6) (xy 71.12 101.6))
     (stroke (width 0) (type default) (color 0 0 0 0))
@@
     (stroke (width 0) (type default) (color 0 0 0 0))
   )
-  (wire (pts (xy 176.53 106.68) (xy 173.99 106.68))
+  (wire (pts (xy 173.99 106.68) (xy 186.69 106.68))
     (stroke (width 0) (type default) (color 0 0 0 0))
   )
@@
     (stroke (width 0) (type default) (color 0 0 0 0))
   )
-  (wire (pts (xy 176.53 102.87) (xy 176.53 106.68))
-    (stroke (width 0) (type default) (color 0 0 0 0))
-  )
   (wire (pts (xy 121.92 71.12) (xy 121.92 99.06))
     (stroke (width 0) (type default) (color 0 0 0 0))
@@
     (stroke (width 0) (type default) (color 0 0 0 0))
   )
-  (wire (pts (xy 186.69 102.87) (xy 186.69 115.57))
+  (wire (pts (xy 186.69 102.87) (xy 186.69 106.68))
     (stroke (width 0) (type default) (color 0 0 0 0))
   )
@@
     (stroke (width 0) (type default) (color 0 0 0 0))
   )
+  (wire (pts (xy 186.69 106.68) (xy 186.69 115.57))
+    (stroke (width 0) (type default) (color 0 0 0 0))
+  )
   (wire (pts (xy 72.39 99.06) (xy 121.92 99.06))
     (stroke (width 0) (type default) (color 0 0 0 0))
@@
     (stroke (width 0) (type default) (color 0 0 0 0))
   )
+  (wire (pts (xy 173.99 99.06) (xy 181.61 99.06))
+    (stroke (width 0) (type default) (color 0 0 0 0))
+  )
   (wire (pts (xy 222.25 102.87) (xy 219.71 102.87))
     (stroke (width 0) (type default) (color 0 0 0 0))
+  )
+  (text "the 120 should be connected at \nthe master device and the last slave one"
+    (at 196.85 90.17 0)
+    (effects (font (size 1.27 1.27)) (justify left bottom))
   )
   (label "B" (at 208.28 102.87 180)
@@
     (in_bom yes) (on_board yes)
     (property "Reference" "R14" (id 0) (at 191.77 83.9216 90))
-    (property "Value" "120" (id 1) (at 191.77 86.233 90))
+    (property "Value" "120NC" (id 1) (at 191.77 86.233 90))
     (property "Footprint" "Resistor_SMD:R_0805_2012Metric_Pad1.15x1.40mm_HandSolder" (id 2) (at 191.77 88.9 0)
       (effects (font (size 1.27 1.27)) hide)

Commit message: Add files via upload
Connections:
- net A renamed RS485+
- net B renamed RS485-
Changed lines of the file:
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@@
     (effects (font (size 1.27 1.27)) (justify left bottom))
   )
-  (label "B" (at 208.28 102.87 180)
+  (label "RS485+" (at 219.71 102.87 180)
     (effects (font (size 1.27 1.27)) (justify right bottom))
   )
-  (label "A" (at 208.28 100.33 180)
+  (label "RS485-" (at 219.71 100.33 180)
     (effects (font (size 1.27 1.27)) (justify right bottom))
   )
-  (label "A" (at 219.71 102.87 0)
-    (effects (font (size 1.27 1.27)) (justify left bottom))
+  (label "RS485-" (at 208.28 102.87 180)
+    (effects (font (size 1.27 1.27)) (justify right bottom))
   )
-  (label "B" (at 219.71 100.33 0)
-    (effects (font (size 1.27 1.27)) (justify left bottom))
+  (label "RS485+" (at 208.28 100.33 180)
+    (effects (font (size 1.27 1.27)) (justify right bottom))
   )
   (global_label "RX" (shape input) (at 66.04 95.25 180) (fields_autoplaced)
