File: iot master.kicad_pcb (KiCad board)
At the start: 2 copper layers, 95.3 x 95.7 mm, 57 parts, among them J1 Screw_Terminal_01x03, J2 Screw_Terminal_01x02, J3 Screw_Terminal_01x03, J4 Screw_Terminal_01x03, J5 Screw_Terminal_01x03, J6 Screw_Terminal_01x03, J7 Screw_Terminal_01x03, J8 Screw_Terminal_01x03, K1 SRD-05VDC-SL-C, K2 SRD-05VDC-SL-C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

Commit message: Add files via upload
Parts:
- R14: value 120 -> 120NC
- R15, R16: value 1k -> 330R
- moved U3 18.8 mm to (145.8, 82.2)
- moved R15 6.49 mm to (117.9, 90.6), turned to -90 degrees
- moved R16 5.42 mm to (115.7, 88.6)
- moved Q3 5.22 mm to (145.3, 64.1)
- moved C3 2.99 mm to (126.1, 86.1), turned to 0 degrees
- moved D3 2.26 mm to (118.0, 86.1), turned to 90 degrees
- moved D2 1.23 mm to (121.6, 91.5), turned to 0 degrees
- moved R13 0.42 mm to (165.3, 60.5)
Routing:
- net +3V3: track 116.9 -> 94.0 mm
- net /relays/RELAY2: track 41.9 -> 63.7 mm
- net /relays/RELAY3: track 27.2 -> 47.8 mm
- net /relays/RELAY4: track 18.4 -> 38.7 mm
- net /relays/RELAY1: track 13.0 -> 33.0 mm
- net GPIO11: track 47.0 -> 30.0 mm
- net GPIO10: track 43.5 -> 27.8 mm
- net GPIO13: track 41.5 -> 25.8 mm
- net GPIO12: track 38.7 -> 23.9 mm
- net GPIO14: track 35.2 -> 21.5 mm
- net GPIO16: track 32.8 -> 19.3 mm
- net +5V: track 182.3 -> 194.2 mm
- net Net-(R5-Pad2): track 8.71 -> 16.4 mm
- net /relays/RELAY6: track 47.3 -> 41.6 mm
- net /relays/RELAY5: track 34.8 -> 29.8 mm
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Other:
- board text added: "D+"
- board text added: "D-"
- board text added: "NC"
- board text removed: "PINS GND----GND GPIO0---D3 VCC----VCC RST----RST TXD----TXD RXD----RXD are exposed for programming the ESP812-E with the node mcu"

Commit message: Add files via upload
Connections:
- net /MAX485CIRCUIT/A renamed /MAX485CIRCUIT/RS485+
- net /MAX485CIRCUIT/B renamed /MAX485CIRCUIT/RS485-
Routing:
- net /MAX485CIRCUIT/RS485-: track 36.1 -> 39.1 mm
- net /MAX485CIRCUIT/RS485+: track 36.9 -> 38.5 mm
- net GND: vias 28 -> 22
